File: kicad/816-v2/816-v2.kicad_sch (KiCad schematic)
At the start: 15 parts, among them J5 EXT, U1 W65C816SxP, U2 74AC74, U3 74AC573, U4 74AC245, U5 ATF22LV10C, U6 ATF22LV10C, Y1 1MHz

Commit message: Update KiCad files to get ready for PCB design
Parts:
- removed C10: 0.1uF, Capacitor_THT:C_Disc_D4.3mm_W1.9mm_P5.00mm, symbol Device:C
- removed J5: EXT, Connector_PinHeader_2.54mm:PinHeader_2x16_P2.54mm_Vertical, symbol Connector:Conn_01x32_Pin
- removed U5, U6: ATF22LV10C, Package_DIP:DIP-24_W7.62mm_Socket, symbol New_Library:ATF22LV10C
- added U5: ATF1504AS-10JU44, Package_LCC:PLCC-44_THT-Socket, symbol custom:ATF1504AS-10JU44
- U2: value 74AC74 -> 74HC74
- U3: value 74AC573 -> 74HC573
- U4: value 74AC245 -> 74HC245
- Y1: value 1MHz -> 8MHz
Connections:
- net A10: now also U5.20 (A10)
- net A11: now also U5.19 (A11)
- net A12: now also U5.18 (A12)
- net A13: now also U5.17 (A13)
- net A14: now also U5.16 (A14)
- net A15: now also U5.14 (A15)
- net A16: now also U5.11 (B0)
- net A17: now also U5.9 (B1)
- net A18: now also U5.8 (B2)
- net A19: now also U5.6 (B3)
- net A20: now also U5.5 (B4)
- net A21: now also U5.4 (B5)
- net A22: now also U5.2 (B6)
- net A23: now also U5.1 (B7)
- net A4: now also U5.28 (A4)
- net A5: now also U5.27 (A5)
- net A6: now also U5.26 (A6)
- net A7: now also U5.25 (A7)
- net A8: now also U5.24 (A8)
- net A9: now also U5.21 (A9)
- net GND: now also U5.10 (GND), U5.22 (GND), U5.30 (GND), U5.42 (GND)
- net IO1CS: now also U5.33 (IO1CS)
- net IO2CS: now also U5.34 (IO2CS)
- net IO3CS: now also U5.36 (IO3CS)
- net IO4CS: now also U5.37 (IO4CS)
- net OE: now also U5.40 (OE)
- net PH2: now also U5.43 (PH2)
- net RAMCS: now also U5.31 (RAMCS)
- net ROMCS: now also U5.29 (ROMCS)
- net RWB: now also U5.44 (RWB)
- net VCC: now also U5.15 (VCC), U5.23 (VCC), U5.3 (VCC), U5.35 (VCC)
- net VDA: now also U5.12 (VDA)
- net WE: now also U5.41 (WE)
- new net IO5CS: U5.39 (IO5CS)
- no-connect marks 17 -> 15
Other:
- added sheet VGA (vga.kicad_sch)

Commit message: Update KiCad files
Parts:
- removed RN1: 10k, Resistor_THT:R_Array_SIP8, symbol Device:R_Network07
- added H1, H2, H3, H4: MountingHole, MountingHole:MountingHole_2.2mm_M2, symbol Mechanical:MountingHole
- added R8, R9: 10k, Resistor_THT:R_Axial_DIN0207_L6.3mm_D2.5mm_P7.62mm_Horizontal, symbol Device:R
Connections:
- net A10: now also U5.17 (A10); no longer U5.20 (A10)
- net A11: now also U5.16 (A11); no longer U5.19 (A11)
- net A12: now also U5.14 (A12); no longer U5.18 (A12)
- net A13: now also U5.12 (A13); no longer U5.17 (A13)
- net A14: now also U5.11 (A14); no longer U5.16 (A14)
- net A15: now also U5.5 (A15); no longer U5.14 (A15)
- net A16: now also U5.33 (B0); no longer U5.11 (B0)
- net A17: now also U5.34 (B1); no longer U5.9 (B1)
- net A18: now also U5.36 (B2); no longer U5.8 (B2)
- net A19: now also U5.37 (B3); no longer U5.6 (B3)
- net A20: now also U5.39 (B4); no longer U5.5 (B4)
- net A21: now also U5.41 (B5); no longer U5.4 (B5)
- net A22: now also U5.40 (B6); no longer U5.2 (B6)
- net A23: now also U5.43 (B7); no longer U5.1 (B7)
- net A4: now also U5.24 (A4); no longer U5.28 (A4)
- net A5: now also U5.25 (A5); no longer U5.27 (A5)
- net A6: now also U5.20 (A6); no longer U5.26 (A6)
- net A7: now also U5.21 (A7); no longer U5.25 (A7)
- net A8: now also U5.18 (A8); no longer U5.24 (A8)
- net A9: now also U5.19 (A9); no longer U5.21 (A9)
- net IO1CS: now also U5.4 (IO1CS); no longer U5.33 (IO1CS)
- net IO2CS: now also U5.6 (IO2CS); no longer U5.34 (IO2CS)
- net IO3CS: now also U5.8 (IO3CS); no longer U5.36 (IO3CS)
- net IO4CS: now also U5.31 (IO4CS); no longer U5.37 (IO4CS)
- net IO5CS: now also U5.9 (IO5CS); no longer U5.39 (IO5CS)
- net IRQB: now also R9.2
- net OE: now also U5.26 (OE); no longer U5.40 (OE)
- net PH2: now also U5.1 (PH2); no longer U5.43 (PH2)
- net RAMCS: now also U5.29 (RAMCS); no longer U5.31 (RAMCS)
- net RESB: now also R8.2
- net ROMCS: now also U5.28 (ROMCS); no longer U5.29 (ROMCS)
- net VCC: now also U1.3 (~{ABORT}), U1.36 (BE), U1.6 (~{NMI}), U2.1 (~{R}), U2.4 (~{S}), R8.1, R9.1
- net VDA: now also U5.2 (VDA); no longer U5.12 (VDA)
- net WE: now also U5.27 (WE); no longer U5.41 (WE)
- no-connect marks 15 -> 13

Commit message: Update KiCad files new pcb revision, hopefully working
Parts:
- H1, H2, H3, H4: footprint MountingHole:MountingHole_2.2mm_M2 -> MountingHole:MountingHole_3.2mm_M3
- U1: value W65C816SxP -> W65C816
- U5: value ATF1504AS-10JU44 -> ATF1504AS
Connections:
- net IO5CS is gone; now on net A14: U5.9 (A14)
- net WE is gone; now on net A23: U5.27 (A23)
- net A10: now also U5.16 (A10); no longer U5.17 (A10)
- net A11: now also U5.14 (A11); no longer U5.16 (A11)
- net A12: now also U5.12 (A12); no longer U5.14 (A12)
- net A13: now also U5.11 (A13); no longer U5.12 (A13)
- net A14: no longer U5.11 (A14)
- net A15: now also U5.1 (A15); no longer U5.5 (A15)
- net A16: now also U5.43 (A16); no longer U5.33 (B0)
- net A17: now also U5.40 (A17); no longer U5.34 (B1)
- net A18: now also U5.41 (A18); no longer U5.36 (B2)
- net A19: now also U5.39 (A19); no longer U5.37 (B3)
- net A20: now also U5.36 (A20); no longer U5.39 (B4)
- net A21: now also U5.37 (A21); no longer U5.41 (B5)
- net A22: now also U5.34 (A22); no longer U5.40 (B6)
- net A23: no longer U5.43 (B7)
- net A4: now also U5.25 (A4); no longer U5.24 (A4)
- net A5: now also U5.20 (A5); no longer U5.25 (A5)
- net A6: now also U5.21 (A6); no longer U5.20 (A6)
- net A7: now also U5.18 (A7); no longer U5.21 (A7)
- net A8: now also U5.19 (A8); no longer U5.18 (A8)
- net A9: now also U5.17 (A9); no longer U5.19 (A9)
- net GND: now also C14.1, C9.1; no longer C14.2, C9.2
- net PH2: now also U5.5 (PH2); no longer U5.1 (PH2)
- net VCC: now also C14.2, C9.2; no longer C14.1, C9.1
- net IO1CS renamed ~{IO2CS}
- net IO2CS renamed ~{IO1CS}
- net IO3CS renamed ~{IO3CS}
- net IO4CS renamed ~{IO4CS}
- net IRQB renamed ~{IRQ}
- net OE renamed ~{OE}
- net PH2B renamed ~{PH2}
- net RAMCS renamed ~{ROMCS}
- net RESB renamed ~{RES}
- net ROMCS renamed ~{RAMCS}
- net RWB renamed R/~{W}
- new net ~{IO5CS}: U5.24 (IO5CS)
- new net ~{WE}: U5.33 (WE)
Other:
- moved on the sheet: C11, C12, C13, C14, C9, H1, H2, R8
