File: kicad/816-v2/untitled.kicad_sch (KiCad schematic)
At the start: 4 parts, among them U13 AS6C4008-55PCN, U8 SST39SF020

Commit message: Update KiCad files new pcb revision, hopefully working
Parts:
- U13: value AS6C4008-55PCN -> AS6C4008; symbol Memory_RAM:AS6C4008-55PCN -> custom:AS6C4008
- U8: symbol Memory_Flash:SST39SF020 -> custom:SST39SF020
Connections:
- net A13: no longer U8.28 (A13)
- net A14: no longer U8.29 (A14)
- net A15: no longer U8.3 (A15)
- net GND: now also U8.28 (A13), U8.29 (A14), U8.3 (A15)
- net OE renamed ~{OE}
- net RAMCS renamed ~{RAMCS}
- net ROMCS renamed ~{ROMCS}
- net WE renamed ~{WE}
Other:
- moved on the sheet: C7, C8

Commit message: Update KiCad files to reflect ROM WE bodge
Connections:
- net VCC: now also U8.31 (PGM)
- no-connect marks 2 -> 1
Changed lines of the file:
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@@
 		(at 166.37 110.49)
-	)
-	(no_connect
-		(at 166.37 115.57)
 	)
 	(bus_entry
@@
 					(unit 1)
 				)
+			)
+		)
+	)
+	(symbol
+		(lib_id "power:VCC")
+		(at 166.37 115.57 0)
+		(unit 1)
+		(exclude_from_sim no)
+		(in_bom yes)
+		(on_board yes)
+		(dnp no)
+		(fields_autoplaced yes)
+		(property "Reference" "#PWR071"
+			(at 166.37 119.38 0)
+			(effects
+				(font
+					(size 1.27 1.27)
+				)
+				(hide yes)
+			)
+		)
+		(property "Value" "VCC"
+			(at 166.37 110.49 0)
+			(effects
+				(font
+					(size 1.27 1.27)
+				)
+				(hide yes)
+			)
+		)
+		(property "Footprint" ""
+			(at 166.37 115.57 0)
+			(effects
+				(font
+					(size 1.27 1.27)
+				)
+				(hide yes)
+			)
+		)
+		(property "Datasheet" ""
+			(at 166.37 115.57 0)
+			(effects
+				(font
+					(size 1.27 1.27)
+				)
+				(hide yes)
+			)
+		)
+		(property "Description" "Power symbol creates a global label with name \"VCC\""
+			(at 166.37 115.57 0)
+			(effects
+				(font
+					(size 1.27 1.27)
+				)
+				(hide yes)
+			)
+		)
+		(pin "1"
+		)
+		(instances
+			(project ""
+				(path "/58394049-29b8-4f07-ad62-86008e573e13/8d99350d-4837-4fef-bdc1-612ee6f0c182"
+					(reference "#PWR071")
+					(unit 1)
+				)
