File: kicad/816-v2/vga.kicad_sch (KiCad schematic)
At the start: 7 parts, among them J7 Pico left, J8 Pico right, J9 DE15_Pins_HighDensity_Mountin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

Commit message: Update KiCad files new pcb revision, hopefully working
Parts:
- J9: value DE15_Pins_HighDensity_MountingHoles -> DE-15 HD; symbol Connector:DE15_Pins_HighDensity_MountingHoles -> custom:DE15_Pins_HighDensity_MountingHoles
Connections:
- net GND: no longer J9.0
- net A0: no longer names the net of J7.19 (Pin_19)
- net A1: no longer names the net of J7.20 (Pin_20)
- net IO4CS renamed ~{IO4CS}
- net RESB renamed ~{RES}
- net RWB renamed R/~{W}
- no-connect marks 16 -> 18
Other:
- note added: "Pi Pico 2"
- moved on the sheet: R1, R3, R4, R5

Commit message: Update KiCad files to reflect ROM WE bodge
Connections:
- net GND: no longer J7.18 (Pin_18), J7.3 (Pin_3), J7.8 (Pin_8), J8.13 (Pin_13), J8.18 (Pin_18), J8.3 (Pin_3), J8.8 (Pin_8)
- net ~{RES}: no longer names the net of J8.12 (Pin_12)
- no-connect marks 18 -> 26
